Commit message: Add files via upload

File: scorbot/urdf/scorbot_description.urdf (robot description, URDF)
Before this commit: robot scorbot, 7 links, 6 joints
Links:
- removed link end_effector
- added link link_5, mass 0.51992001; collision mesh filename=package://scorbot/meshes/link_5.stl scale=0.001 0.001 0.001; visual mesh filename=package://scorbot/meshes/link_5.stl scale=0.001 0.001 0.001
Joints:
- removed joint tool
- added joint j5: type revolute, parent link_4, child link_5, origin xyz=0.1319 0.0 0.0 rpy=0.0 0.0 0.0, axis 1.0 0.0 0.0, limit lower=-3.14 upper=3.14 effort=10.0 velocity=20.0
- joint j2: limit lower=0.0 upper=3.14 effort=10.0 velocity=20.0 -> lower=-3.14 upper=3.14 effort=10.0 velocity=20.0
- joint j3: limit lower=0.0 upper=3.14 effort=10.0 velocity=20.0 -> lower=-3.14 upper=3.14 effort=10.0 velocity=20.0
- joint j4: limit lower=0.0 upper=3.14 effort=10.0 velocity=20.0 -> lower=-3.14 upper=3.14 effort=10.0 velocity=20.0
